File: pcb/BlinkyBall-switchedcap.brd (EAGLE design)
At the start: 18 x 18 mm, 21 parts, among them U1 Tiny85-20-SMT

Commit message: RevC pcb design: rounded rect, switch IR pinout, space out test points
Parts:
- C2, C3, C4: value 100nF -> 2.2uF
- renumbered LED_BOT to D1, LED_TOP to D2, U$2 to U$1
Changed lines of the file:
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@@
 <layer number="17" name="Pads" color="2" fill="1" visible="yes" active="yes"/>
 <layer number="18" name="Vias" color="2" fill="1" visible="yes" active="yes"/>
-<layer number="19" name="Unrouted" color="6" fill="1" visible="yes" active="yes"/>
+<layer number="19" name="Unrouted" color="6" fill="1" visible="no" active="yes"/>
 <layer number="20" name="Dimension" color="15" fill="1" visible="yes" active="yes"/>
 <layer number="21" name="tPlace" color="7" fill="1" visible="yes" active="yes"/>
@@
 </autorouter>
 <elements>
-<element name="U$2" library="blinkinlabs" package="BATTERY_COVER_AG3" value="BATTERY_BUTTON_CELLAG3" x="9" y="9" rot="MR270"/>
+<element name="U$1" library="blinkinlabs" package="BATTERY_COVER_AG3" value="BATTERY_BUTTON_CELLAG3" x="9" y="9" rot="MR270"/>
 <element name="U1" library="SparkFun-DigitalIC" package="SO08-EIAJ" value="Tiny85-20-SMT" x="9" y="9.5" smashed="yes" rot="R270">
 <attribute name="PROD_ID" value="IC-09092" x="9" y="9.5" size="1.778" layer="27" rot="R270" display="off"/>
@@
 <element name="TP5" library="SparkFun-Passives" package="PAD.03X.05" value="TEST-POINT3X5" x="12.7" y="15.8"/>
 <element name="TP6" library="SparkFun-Passives" package="PAD.03X.05" value="TEST-POINT3X5" x="3.3" y="11.2"/>
-<element name="LED_BOT" library="adafruit" package="LED5MM" value="" x="9" y="2.2" smashed="yes" rot="MR0">
+<element name="D1" library="adafruit" package="LED5MM" value="" x="9" y="2.2" smashed="yes" rot="MR0">
 <attribute name="VALUE" x="5.7996" y="0.3966" size="1.27" layer="28" ratio="10" rot="MR0"/>
 </element>
-<element name="LED_TOP" library="adafruit" package="LED5MM" value="" x="9" y="15.8" smashed="yes" rot="MR180">
+<element name="D2" library="adafruit" package="LED5MM" value="" x="9" y="15.8" smashed="yes" rot="MR180">
 <attribute name="VALUE" x="12.2004" y="17.6034" size="1.27" layer="28" ratio="10" rot="MR180"/>
 </element>
@@
 <element name="U$3" library="blinkinlabs" package="SW-18015P" value="SW-18015P" x="2" y="9" rot="MR270"/>
 <element name="U$4" library="blinkinlabs" package="SOT23-6" value="REG71050" x="13" y="5.5" rot="R270"/>
-<element name="C2" library="adafruit" package="C0603" value="100nF" x="15.6" y="5.5" rot="R270"/>
-<element name="C3" library="adafruit" package="C0603" value="100nF" x="8.7" y="6.1"/>
-<element name="C4" library="adafruit" package="C0603" value="100nF" x="13" y="3"/>
+<element name="C2" library="adafruit" package="C0603" value="2.2uF" x="15.6" y="5.5" rot="R270"/>
+<element name="C3" library="adafruit" package="C0603" value="2.2uF" x="8.7" y="6.1"/>
+<element name="C4" library="adafruit" package="C0603" value="2.2uF" x="13" y="3"/>
 </elements>
 <signals>
@@
 <contactref element="R4" pad="2"/>
 <contactref element="TP4" pad="P$1"/>
-<contactref element="U$2" pad="+3"/>
-<contactref element="U$2" pad="+2"/>
-<contactref element="U$2" pad="+1"/>
-<contactref element="U$2" pad="+4"/>
+<contactref element="U$1" pad="+3"/>
+<contactref element="U$1" pad="+2"/>
+<contactref element="U$1" pad="+1"/>
+<contactref element="U$1" pad="+4"/>
 <contactref element="C1" pad="1"/>
 <contactref element="U1" pad="8"/>
@@
 </signal>
 <signal name="GND">
-<contactref element="U$2" pad="-"/>
+<contactref element="U$1" pad="-"/>
 <contactref element="U1" pad="4"/>
 <contactref element="C1" pad="2"/>
@@
 <via x="15" y="3.5" extent="1-16" drill="0.3"/>
 <wire x1="15" y1="3.5" x2="15.5" y2="4" width="0.4064" layer="16"/>
-<contactref element="LED_BOT" pad="K"/>
-<contactref element="LED_TOP" pad="K"/>
+<contactref element="D1" pad="K"/>
+<contactref element="D2" pad="K"/>
 <wire x1="5.6218" y1="7.595" x2="7.095" y2="7.595" width="0.4064" layer="1"/>
 <wire x1="7.095" y1="7.595" x2="7.3" y2="7.8" width="0.4064" layer="1"/>
@@
 <signal name="N$1">
 <contactref element="R3" pad="1"/>
-<contactref element="LED_TOP" pad="A"/>
+<contactref element="D2" pad="A"/>
 <wire x1="5.6" y1="14.35" x2="6.28" y2="14.35" width="0.4064" layer="1"/>
 <wire x1="6.28" y1="14.35" x2="7.73" y2="15.8" width="0.4064" layer="1"/>
@@
 <signal name="N$2">
 <contactref element="R2" pad="1"/>
-<contactref element="LED_BOT" pad="A"/>
+<contactref element="D1" pad="A"/>
 <wire x1="10.27" y1="2.2" x2="10.27" y2="2.07" width="0.4064" layer="1"/>
 <wire x1="10.27" y1="2.07" x2="9" y2="0.8" width="0.4064" layer="1"/>
