File: pcb/BlinkyBall.brd (EAGLE design)
At the start: 18 x 18 mm, 18 parts, among them U1 Tiny85-20-SMT

Commit message: PCB: Fix referene names
Parts:
- renumbered LED_BOT to D2, LED_TOP to D1, U$1 to U2, U$2 to J2, U$3 to J1, U$5 to U3
Changed lines of the file:
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@@
 <setting verticaltext="up"/>
 </settings>
-<grid distance="0.5" unitdist="mm" unit="mm" style="lines" multiple="1" display="yes" altdistance="0.1" altunitdist="mm" altunit="mm"/>
+<grid distance="0.5" unitdist="mm" unit="mm" style="lines" multiple="1" display="no" altdistance="0.1" altunitdist="mm" altunit="mm"/>
 <layers>
 <layer number="1" name="Top" color="4" fill="1" visible="yes" active="yes"/>
@@
 <layer number="14" name="Route14" color="1" fill="6" visible="no" active="no"/>
 <layer number="15" name="Route15" color="4" fill="6" visible="no" active="no"/>
-<layer number="16" name="Bottom" color="1" fill="1" visible="yes" active="yes"/>
+<layer number="16" name="Bottom" color="1" fill="1" visible="no" active="yes"/>
 <layer number="17" name="Pads" color="2" fill="1" visible="yes" active="yes"/>
 <layer number="18" name="Vias" color="2" fill="1" visible="yes" active="yes"/>
-<layer number="19" name="Unrouted" color="6" fill="1" visible="yes" active="yes"/>
+<layer number="19" name="Unrouted" color="6" fill="1" visible="no" active="yes"/>
 <layer number="20" name="Dimension" color="15" fill="1" visible="yes" active="yes"/>
 <layer number="21" name="tPlace" color="7" fill="1" visible="yes" active="yes"/>
@@
 <layer number="24" name="bOrigins" color="15" fill="1" visible="yes" active="yes"/>
 <layer number="25" name="tNames" color="7" fill="1" visible="yes" active="yes"/>
-<layer number="26" name="bNames" color="7" fill="1" visible="yes" active="yes"/>
+<layer number="26" name="bNames" color="7" fill="1" visible="no" active="yes"/>
 <layer number="27" name="tValues" color="7" fill="1" visible="no" active="yes"/>
 <layer number="28" name="bValues" color="7" fill="1" visible="no" active="yes"/>
@@
 <layer number="45" name="Holes" color="7" fill="1" visible="no" active="yes"/>
 <layer number="46" name="Milling" color="3" fill="1" visible="yes" active="yes"/>
-<layer number="47" name="Measures" color="7" fill="1" visible="yes" active="yes"/>
+<layer number="47" name="Measures" color="7" fill="1" visible="no" active="yes"/>
 <layer number="48" name="Document" color="7" fill="1" visible="yes" active="yes"/>
 <layer number="49" name="Reference" color="7" fill="1" visible="no" active="yes"/>
@@
 </autorouter>
 <elements>
-<element name="U$2" library="blinkinlabs" package="BATTERY_COVER_AG3" value="BATTERY_BUTTON_CELLAG3" x="9" y="9" rot="MR270"/>
+<element name="J2" library="blinkinlabs" package="BATTERY_COVER_AG3" value="BATTERY_BUTTON_CELLAG3" x="9" y="9" rot="MR270"/>
 <element name="U1" library="SparkFun-DigitalIC" package="SO08-EIAJ" value="Tiny85-20-SMT" x="9.7" y="9.5" smashed="yes" rot="R270">
 <attribute name="PROD_ID" value="IC-09092" x="9.7" y="9.5" size="1.778" layer="27" rot="R270" display="off"/>
 </element>
 <element name="C1" library="adafruit" package="C0603" value="100nF" x="12.1" y="13.5" smashed="yes" rot="R90"/>
-<element name="U$5" library="blinkinlabs" package="TSOP321" value="TSOP321" x="3.3" y="4" rot="MR45"/>
+<element name="U3" library="blinkinlabs" package="TSOP321" value="TSOP321" x="3.3" y="4" rot="MR45"/>
 <element name="R2" library="adafruit" package="R0603" value="10" x="13" y="3" smashed="yes" rot="R180"/>
 <element name="R3" library="adafruit" package="R0603" value="10" x="5.6" y="13.5" smashed="yes" rot="R90"/>
@@
 <element name="TP5" library="SparkFun-Passives" package="PAD.03X.05" value="TEST-POINT3X5" x="4.2" y="8"/>
 <element name="TP6" library="SparkFun-Passives" package="PAD.03X.05" value="TEST-POINT3X5" x="4.2" y="11.2"/>
-<element name="LED_BOT" library="adafruit" package="LED5MM" value="" x="9" y="2.2" smashed="yes" rot="MR180">
+<element name="D2" library="adafruit" package="LED5MM" value="" x="9" y="2.2" smashed="yes" rot="MR180">
 <attribute name="VALUE" x="12.2004" y="4.0034" size="1.27" layer="28" ratio="10" rot="MR180"/>
 </element>
-<element name="LED_TOP" library="adafruit" package="LED5MM" value="" x="9" y="15.8" smashed="yes" rot="MR0">
+<element name="D1" library="adafruit" package="LED5MM" value="" x="9" y="15.8" smashed="yes" rot="MR0">
 <attribute name="VALUE" x="5.7996" y="13.9966" size="1.27" layer="28" ratio="10" rot="MR0"/>
 </element>
-<element name="U$1" library="blinkinlabs" package="SOT23" value="AO3418" x="13.4" y="5.5" smashed="yes" rot="R90">
+<element name="U2" library="blinkinlabs" package="SOT23" value="AO3418" x="13.4" y="5.5" smashed="yes" rot="R90">
 <attribute name="VALUE" x="16.575" y="3.595" size="1.27" layer="27" rot="R90"/>
 </element>
@@
 <attribute name="VALUE" x="12.168" y="14.389" size="1.27" layer="27" rot="R270"/>
 </element>
-<element name="U$3" library="blinkinlabs" package="SW-18015P" value="SW-18015P" x="2" y="9" rot="MR90"/>
+<element name="J1" library="blinkinlabs" package="SW-18015P" value="SW-18015P" x="2" y="9" rot="MR90"/>
 </elements>
 <signals>
@@
 <contactref element="R4" pad="2"/>
 <contactref element="TP4" pad="P$1"/>
-<contactref element="U$2" pad="+3"/>
-<contactref element="U$2" pad="+2"/>
-<contactref element="U$2" pad="+1"/>
-<contactref element="U$2" pad="+4"/>
+<contactref element="J2" pad="+3"/>
+<contactref element="J2" pad="+2"/>
+<contactref element="J2" pad="+1"/>
+<contactref element="J2" pad="+4"/>
 <contactref element="C1" pad="1"/>
 <contactref element="U1" pad="8"/>
-<contactref element="LED_TOP" pad="A"/>
-<contactref element="LED_BOT" pad="A"/>
+<contactref element="D1" pad="A"/>
+<contactref element="D2" pad="A"/>
 <wire x1="10.27" y1="15.8" x2="10.27" y2="13.77" width="0.4064" layer="1"/>
 <wire x1="10.27" y1="13.77" x2="10" y2="13.5" width="0.4064" layer="1"/>
@@
 </signal>
 <signal name="GND">
-<contactref element="U$2" pad="-"/>
+<contactref element="J2" pad="-"/>
 <contactref element="U1" pad="4"/>
 <contactref element="C1" pad="2"/>
@@
 <vertex x="0" y="18"/>
 </polygon>
-<contactref element="U$1" pad="2"/>
+<contactref element="U2" pad="2"/>
 <contactref element="R1" pad="1"/>
 <wire x1="14.5" y1="6.45" x2="15.75" y2="6.45" width="0.4064" layer="1"/>
@@
 <wire x1="6.3218" y1="7.595" x2="4.2" y2="7.595" width="0.4064" layer="1"/>
 <wire x1="4.2" y1="8" x2="4.2" y2="7.595" width="0.4064" layer="1"/>
-<contactref element="U$5" pad="P$2"/>
-<contactref element="U$3" pad="P$1"/>
+<contactref element="U3" pad="P$2"/>
+<contactref element="J1" pad="P$1"/>
 <wire x1="4.1" y1="9.4" x2="4.1" y2="8.1" width="0.4064" layer="1"/>
 <wire x1="4.1" y1="8.1" x2="4.2" y2="8" width="0.4064" layer="1"/>
@@
 <wire x1="3.5" y1="12.65" x2="2.85" y2="12.65" width="0.4064" layer="1"/>
 <wire x1="2.85" y1="12.65" x2="2" y2="11.8" width="0.4064" layer="1"/>
-<contactref element="U$3" pad="P$2"/>
+<contactref element="J1" pad="P$2"/>
 <wire x1="2" y1="11.8" x2="2" y2="10.75" width="0.4064" layer="1"/>
 <wire x1="9.1" y1="12" x2="3.25" y2="12" width="0.4064" layer="16"/>
@@
 <contactref element="U1" pad="6"/>
 <contactref element="TP2" pad="P$1"/>
-<contactref element="U$1" pad="1"/>
+<contactref element="U2" pad="1"/>
 <contactref element="R1" pad="2"/>
 <wire x1="13.0528" y1="8.865" x2="15.065" y2="8.865" width="0.4064" layer="1"/>
@@
 <wire x1="7.435" y1="8.865" x2="7.9" y2="8.4" width="0.4064" layer="1"/>
 <wire x1="7.9" y1="8.4" x2="7.9" y2="7.1" width="0.4064" layer="1"/>
-<contactref element="U$5" pad="P$3"/>
+<contactref element="U3" pad="P$3"/>
 <wire x1="1.50395" y1="5.79605" x2="2.1" y2="5.2" width="0.4064" layer="1"/>
 <wire x1="2.1" y1="5.2" x2="5.1" y2="5.2" width="0.4064" layer="1"/>
@@
 <wire x1="6.3218" y1="10.135" x2="7.665" y2="10.135" width="0.4064" layer="1"/>
 <wire x1="7.665" y1="10.135" x2="8.6" y2="9.2" width="0.4064" layer="1"/>
-<contactref element="U$5" pad="P$1"/>
+<contactref element="U3" pad="P$1"/>
 <wire x1="5.1" y1="4.1" x2="5.1" y2="2.3" width="0.4064" layer="1"/>
 <wire x1="5.1" y1="4.1" x2="7" y2="6" width="0.4064" layer="1"/>
@@
 </signal>
 <signal name="N$2">
-<contactref element="LED_BOT" pad="K"/>
+<contactref element="D2" pad="K"/>
 <contactref element="R2" pad="2"/>
 <wire x1="12.15" y1="3" x2="11.07" y2="3" width="0.4064" layer="1"/>
@@
 </signal>
 <signal name="N$3">
-<contactref element="LED_TOP" pad="K"/>
+<contactref element="D1" pad="K"/>
 <contactref element="R3" pad="2"/>
 <wire x1="7.73" y1="15.8" x2="6.3" y2="15.8" width="0.4064" layer="1"/>
@@
 <signal name="N$4">
 <contactref element="R2" pad="1"/>
-<contactref element="U$1" pad="3"/>
+<contactref element="U2" pad="3"/>
 <contactref element="R3" pad="1"/>
 <wire x1="13.85" y1="3" x2="13.85" y2="3.15" width="0.4064" layer="1"/>

Commit message: Correct pinout for IR receiver
Connections:
- net IR_ENABLE renamed IR_POWER
- net IR_SIGNAL renamed IR_DATA
- net LED_TOP renamed LED_ON
Changed lines of the file:
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@@
 <layer number="14" name="Route14" color="1" fill="6" visible="no" active="no"/>
 <layer number="15" name="Route15" color="4" fill="6" visible="no" active="no"/>
-<layer number="16" name="Bottom" color="1" fill="1" visible="no" active="yes"/>
+<layer number="16" name="Bottom" color="1" fill="1" visible="yes" active="yes"/>
 <layer number="17" name="Pads" color="2" fill="1" visible="yes" active="yes"/>
 <layer number="18" name="Vias" color="2" fill="1" visible="yes" active="yes"/>
@@
 <wire x1="3.25" y1="12" x2="2" y2="10.75" width="0.4064" layer="16"/>
 </signal>
-<signal name="LED_TOP">
+<signal name="LED_ON">
 <contactref element="U1" pad="6"/>
 <contactref element="TP2" pad="P$1"/>
@@
 <wire x1="15.395" y1="7.595" x2="15.8" y2="8" width="0.4064" layer="1"/>
 </signal>
-<signal name="IR_ENABLE">
+<signal name="IR_POWER">
 <contactref element="U1" pad="3"/>
 <wire x1="6.3218" y1="8.865" x2="7.435" y2="8.865" width="0.4064" layer="1"/>
@@
 <wire x1="6.6" y1="6.7" x2="5.1" y2="5.2" width="0.4064" layer="1"/>
 </signal>
-<signal name="IR_SIGNAL">
+<signal name="IR_DATA">
 <contactref element="U1" pad="2"/>
 <wire x1="6.3218" y1="10.135" x2="7.665" y2="10.135" width="0.4064" layer="1"/>
